File: kicad/VeloDashboard/VeloDashboard.kicad_sch (KiCad schematic)
At the start: 42 parts, among them IC1 LDD-700L, IC2 LDD-700L, IC3 LDD-700L, IC4 LDD-700L, J1 Speed Sensor, J1.out Polulu Power, J2 OLED 128 x 64, K1 HF3-03, Q1 IRF520, Q2 BC546, SW1 On / Off switch, SW2 Down (lights), SW3 Left, SW4 Up (lights), SW5 Horn, SW6 Display, SW7 Right, SW8 Brake, U1 SN74AHCT125N, U2 LC78_05 2.0

Commit message: pcb cleanup
Parts:
- removed BZ1: Buzzer, symbol Device:Buzzer
- removed D1: D, symbol Device:D
- removed HORN: (no value), symbol Device:Buzzer
- removed K1: HF3-03, Relay_SMD:Relay_SPDT_AXICOM_HF3Series_75ohms_Pitch1.27mm, symbol Relay:HF3-03
- removed Q1: IRF520, TO270P460X1020X2008-3P, symbol IRF520:IRF520
- removed Q2: BC546, Package_TO_SOT_THT:TO-92_Inline, symbol Transistor_BJT:BC546
- removed R14: 10k, symbol Device:R
- removed R15: 1k, symbol Device:R
- gave numbers to parts that had none: 1
- renumbered J1.in to J1.in1, J1.out to J1.out1
Connections:
- net GND1 is gone; now on net GND: IC1.4 (-VIN), IC2.4 (-VIN), IC3.4 (-VIN), IC4.4 (-VIN)
- net GND: now also J2.2 (Pin_2), U3.32 (GND)
- net +3.3V: now reaches BT1.1 (+), U3.15 (VBAT)
- no-connect marks 41 -> 45
Other:
- moved on the sheet: C1, IC1, IC2, IC3, IC4, J1.in1, J1.out1, J2, R1, R2, R3, R4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
