File: kicad/VeloDashboard/VeloDashboard.kicad_sch (KiCad schematic)
At the start: 58 parts, among them IC1 LDD-700L, IC2 LDD-700L, IC3 LDD-700L, IC4 LDD-700L, IC5 LDD-700L, IC6 LDD-700L, J1 OLED, J1.out1 Polulu Power, J10 Cadans sensor, J11 Addon 2, J12 extra led strips, J2 LED STRIPS, J3 To Dashboard, J4 To Computer, J5 Speed Sensor, J6 Headlights, J7 Rearlights, J8 Blinkers, J9 PowerSwitch, SW2 Left, SW3 Down (lights), SW4 Up (lights), SW5 Brake, SW6 Horn, SW7 Display, SW8 Right, U1 SN74AHCT125N, U2 LC78_05 2.0, U3 Teensy4.0

Commit message: power adjustments
Parts:
- added C2: 10µF, Capacitor_THT:CP_Radial_D10.0mm_P7.50mm, symbol Device:C_Polarized
- C1: value 22µF -> 470µF
- R21, R22, R23, R24: value 370 -> 470
Connections:
- net +12V: now also C2.1
- net GND: now also C2.2
Other:
- moved on the sheet: R1, R2
Changed lines of the file:
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@@
 	)
 	(junction
-		(at 170.18 88.9)
+		(at 226.06 124.46)
 		(diameter 0)
 		(color 0 0 0 0)
 	)
 	(junction
-		(at 236.22 124.46)
+		(at 170.18 88.9)
 		(diameter 0)
 		(color 0 0 0 0)
@@
 	)
 	(junction
+		(at 237.49 124.46)
+		(diameter 0)
+		(color 0 0 0 0)
+	)
+	(junction
 		(at 36.83 167.64)
 		(diameter 0)
@@
 	)
 	(junction
-		(at 236.22 137.16)
+		(at 237.49 137.16)
 		(diameter 0)
 		(color 0 0 0 0)
 	)
 	(junction
-		(at 229.87 124.46)
+		(at 199.39 107.95)
 		(diameter 0)
 		(color 0 0 0 0)
 	)
 	(junction
-		(at 199.39 107.95)
+		(at 237.49 148.59)
 		(diameter 0)
 		(color 0 0 0 0)
@@
 	)
 	(junction
-		(at 236.22 148.59)
+		(at 226.06 132.08)
 		(diameter 0)
 		(color 0 0 0 0)
@@
 	(wire
 		(pts
-			(xy 236.22 124.46) (xy 243.84 124.46)
-		)
-		(stroke
-			(width 0)
-			(type default)
-		)
-	)
-	(wire
-		(pts
 			(xy 39.37 38.1) (xy 40.64 38.1)
 		)
@@
 	(wire
 		(pts
+			(xy 237.49 124.46) (xy 243.84 124.46)
+		)
+		(stroke
+			(width 0)
+			(type default)
+		)
+	)
+	(wire
+		(pts
 			(xy 21.59 152.4) (xy 21.59 179.07)
 		)
@@
 	(wire
 		(pts
-			(xy 236.22 148.59) (xy 229.87 148.59)
+			(xy 226.06 148.59) (xy 237.49 148.59)
 		)
 		(stroke
@@
 	(wire
 		(pts
-			(xy 236.22 137.16) (xy 237.49 137.16)
+			(xy 237.49 137.16) (xy 238.76 137.16)
 		)
 		(stroke
@@
 	(wire
 		(pts
-			(xy 229.87 124.46) (xy 236.22 124.46)
+			(xy 68.58 53.34) (xy 68.58 69.85)
 		)
 		(stroke
@@
 	(wire
 		(pts
-			(xy 68.58 53.34) (xy 68.58 69.85)
+			(xy 96.52 48.26) (xy 99.06 48.26)
 		)
 		(stroke
@@
 	(wire
 		(pts
-			(xy 96.52 48.26) (xy 99.06 48.26)
+			(xy 90.17 167.64) (xy 92.71 167.64)
 		)
 		(stroke
@@
 	(wire
 		(pts
-			(xy 90.17 167.64) (xy 92.71 167.64)
+			(xy 96.52 45.72) (xy 99.06 45.72)
 		)
 		(stroke
@@
 	(wire
 		(pts
-			(xy 96.52 45.72) (xy 99.06 45.72)
+			(xy 68.58 43.18) (xy 68.58 53.34)
 		)
 		(stroke
@@
 	(wire
 		(pts
-			(xy 68.58 43.18) (xy 68.58 53.34)
+			(xy 86.36 91.44) (xy 86.36 121.92)
 		)
 		(stroke
@@
 	(wire
 		(pts
-			(xy 86.36 91.44) (xy 86.36 121.92)
+			(xy 91.44 96.52) (xy 91.44 116.84)
 		)
 		(stroke
@@
 	(wire
 		(pts
-			(xy 91.44 96.52) (xy 91.44 116.84)
+			(xy 226.06 124.46) (xy 237.49 124.46)
 		)
 		(stroke
@@
 	(wire
 		(pts
-			(xy 236.22 132.08) (xy 236.22 137.16)
+			(xy 237.49 132.08) (xy 237.49 137.16)
 		)
 		(stroke
@@
 	(wire
 		(pts
-			(xy 220.98 124.46) (xy 229.87 124.46)
+			(xy 220.98 124.46) (xy 226.06 124.46)
 		)
 		(stroke
@@
 	(wire
 		(pts
-			(xy 229.87 132.08) (xy 229.87 148.59)
+			(xy 226.06 132.08) (xy 226.06 148.59)
 		)
 		(stroke
@@
 	(wire
 		(pts
-			(xy 254 148.59) (xy 236.22 148.59)
+			(xy 254 148.59) (xy 237.49 148.59)
 		)
 		(stroke
@@
 	(wire
 		(pts
-			(xy 220.98 132.08) (xy 229.87 132.08)
+			(xy 220.98 132.08) (xy 226.06 132.08)
 		)
 		(stroke
@@
 	(wire
 		(pts
-			(xy 236.22 137.16) (xy 236.22 140.97)
+			(xy 237.49 137.16) (xy 237.49 140.97)
 		)
 		(stroke
@@
 	(global_label "Power meter"
 		(shape output)
-		(at 237.49 137.16 0)
+		(at 238.76 137.16 0)
 		(fields_autoplaced yes)
 		(effects
@@
 		)
 		(property "Intersheetrefs" "${INTERSHEET_REFS}"
-			(at 251.5103 137.16 0)
+			(at 252.7803 137.16 0)
 			(effects
 				(font
@@
 	(symbol
 		(lib_id "power:+12V")
-		(at 229.87 124.46 0)
+		(at 237.49 124.46 0)
 		(unit 1)
 		(exclude_from_sim no)
@@
 		(fields_autoplaced yes)
 		(property "Reference" "#PWR08"
-			(at 229.87 128.27 0)
+			(at 237.49 128.27 0)
 			(effects
 				(font
@@
 		)
 		(property "Value" "+12V"
-			(at 229.87 119.38 0)
+			(at 237.49 119.38 0)
 			(effects
 				(font
@@
 		)
 		(property "Footprint" ""
-			(at 229.87 124.46 0)
+			(at 237.49 124.46 0)
 			(effects
 				(font
@@
 		)
 		(property "Datasheet" ""
-			(at 229.87 124.46 0)
+			(at 237.49 124.46 0)
 			(effects
 				(font
@@
 		)
 		(property "Description" "Power symbol creates a global label with name \"+12V\""
-			(at 229.87 124.46 0)
+			(at 237.49 124.46 0)
 			(effects
 				(font
@@
 		(fields_autoplaced yes)
 		(property "Reference" "C1"
-			(at 269.621 129.2773 0)
+			(at 270.51 128.6509 0)
 			(effects
 				(font
@@
 			)
 		)
-		(property "Value" "22µF"
-			(at 269.621 131.1983 0)
+		(property "Value" "470µF"
+			(at 270.51 131.1909 0)
 			(effects
 				(font
@@
 	(symbol
 		(lib_id "Device:R")
-		(at 236.22 128.27 0)
+		(at 237.49 128.27 0)
 		(unit 1)
 		(exclude_from_sim no)
@@
 		(fields_autoplaced yes)
 		(property "Reference" "R1"
-			(at 237.998 127.6263 0)
+			(at 239.268 127.6263 0)
 			(effects
 				(font
@@
 		)
 		(property "Value" "4M"
-			(at 237.998 129.5473 0)
+			(at 239.268 129.5473 0)
 			(effects
 				(font
@@
 		)
 		(property "Footprint" "Resistor_THT:R_Axial_DIN0207_L6.3mm_D2.5mm_P10.16mm_Horizontal"
-			(at 234.442 128.27 90)
+			(at 235.712 128.27 90)
 			(effects
 				(font
@@
 		)
 		(property "Datasheet" "~"
-			(at 236.22 128.27 0)
+			(at 237.49 128.27 0)
 			(effects
 				(font
@@
 		)
 		(property "Description" "Resistor"
-			(at 236.22 128.27 0)
+			(at 237.49 128.27 0)
 			(effects
 				(font
@@
 			)
 		)
-		(property "Value" "370"
+		(property "Value" "470"
 			(at 44.45 55.88 90)
 			(effects
@@
 	(symbol
 		(lib_id "Device:R")
-		(at 236.22 144.78 0)
+		(at 237.49 144.78 0)
 		(unit 1)
 		(exclude_from_sim no)
@@
 		(fields_autoplaced yes)
 		(property "Reference" "R2"
-			(at 237.998 144.1363 0)
+			(at 239.268 144.1363 0)
 			(effects
 				(font
@@
 		)
 		(property "Value" "1M"
-			(at 237.998 146.0573 0)
+			(at 239.268 146.0573 0)
 			(effects
 				(font
@@
 		)
 		(property "Footprint" "Resistor_THT:R_Axial_DIN0207_L6.3mm_D2.5mm_P10.16mm_Horizontal"
-			(at 234.442 144.78 90)
+			(at 235.712 144.78 90)
 			(effects
 				(font
@@
 		)
 		(property "Datasheet" "~"
-			(at 236.22 144.78 0)
+			(at 237.49 144.78 0)
 			(effects
 				(font
@@
 		)
 		(property "Description" "Resistor"
-			(at 236.22 144.78 0)
+			(at 237.49 144.78 0)
 			(effects
 				(font
@@
 			)
 		)
-		(property "Value" "370"
+		(property "Value" "470"
 			(at 44.45 25.4 90)
 			(effects
@@
 			)
 		)
-		(property "Value" "370"
+		(property "Value" "470"
 			(at 44.45 45.72 90)
 			(effects
@@
 	)
 	(symbol
+		(lib_id "Device:C_Polarized")
+		(at 226.06 128.27 0)
+		(unit 1)
+		(exclude_from_sim no)
+		(in_bom yes)
+		(on_board yes)
+		(dnp no)
+		(fields_autoplaced yes)
+		(property "Reference" "C2"
+			(at 229.87 126.1109 0)
+			(effects
+				(font
+					(size 1.27 1.27)
+				)
+				(justify left)
+			)
+		)
+		(property "Value" "10µF"
+			(at 229.87 128.6509 0)
+			(effects
+				(font
+					(size 1.27 1.27)
+				)
+				(justify left)
+			)
+		)
+		(property "Footprint" "Capacitor_THT:CP_Radial_D10.0mm_P7.50mm"
+			(at 227.0252 132.08 0)
+			(effects
+				(font
+					(size 1.27 1.27)
+				)
+				(hide yes)
+			)
+		)
+		(property "Datasheet" "~"
+			(at 226.06 128.27 0)
+			(effects
+				(font
+					(size 1.27 1.27)
+				)
+				(hide yes)
+			)
+		)
+		(property "Description" "Polarized capacitor"
+			(at 226.06 128.27 0)
+			(effects
+				(font
+					(size 1.27 1.27)
+				)
+				(hide yes)
+			)
+		)
+		(pin "1"
+		)
+		(pin "2"
+		)
+		(instances
+			(project "VeloDashboard"
+				(path "/2446985a-a6e1-44ac-a22d-63b6c5e9fbf1"
+					(reference "C2")
+					(unit 1)
+				)
+			)
+		)
+	)
+	(symbol
 		(lib_id "LDD-700L:LDD-700L")
 		(at 243.84 107.95 180)
@@
 			)
 		)
-		(property "Value" "370"
+		(property "Value" "470"
 			(at 44.45 35.56 90)
 			(effects

Commit message: update dasbboard connector on computer
Parts:
- removed J3: To Dashboard, Connector_PinHeader_2.54mm:PinHeader_1x08_P2.54mm_Horizontal, symbol Connector:Conn_01x08_Pin
- added J13: To Dashboard, symbol Connector:Conn_01x06_Pin
Connections:
- net GND: now also J13.6 (Pin_6)
- net at R4.2, R8.1: now also J13.5 (Pin_5)
- net at R10.2: now also J13.2 (Pin_2)
- net at R3.1, R7.1: now also J13.4 (Pin_4)
- net at R5.1, R6.1: now also J13.3 (Pin_3)
- net at R9.2: now also J13.1 (Pin_1)
- no-connect marks 31 -> 29
Changed lines of the file:
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@@
 	)
 	(no_connect
-		(at 154.94 132.08)
-	)
-	(no_connect
 		(at 154.94 50.8)
 	)
@@
 	)
 	(no_connect
-		(at 152.4 132.08)
-	)
-	(no_connect
 		(at 154.94 63.5)
 	)
@@
 	(wire
 		(pts
-			(xy 157.48 129.54) (xy 157.48 132.08)
+			(xy 152.4 129.54) (xy 152.4 132.08)
 		)
 		(stroke
@@
 	(wire
 		(pts
-			(xy 170.18 129.54) (xy 157.48 129.54)
+			(xy 170.18 129.54) (xy 152.4 129.54)
 		)
 		(stroke
@@
 	)
 	(rectangle
-		(start 130.81 132.08)
-		(end 165.1 152.4)
+		(start 132.08 132.08)
+		(end 160.02 149.86)
 		(stroke
 			(width 0)
@@
 	(text "Dashboard connector"
 		(exclude_from_sim no)
-		(at 138.43 148.59 0)
+		(at 135.89 148.59 0)
 		(effects
 			(font
@@
 	)
 	(symbol
-		(lib_id "Connector:Conn_01x08_Pin")
-		(at 147.32 137.16 90)
-		(unit 1)
-		(exclude_from_sim no)
-		(in_bom yes)
-		(on_board yes)
-		(dnp no)
-		(property "Reference" "J3"
-			(at 148.59 138.8317 90)
-			(effects
-				(font
-					(size 1.27 1.27)
-				)
-			)
-		)
-		(property "Value" "To Dashboard"
-			(at 148.59 140.7527 90)
-			(effects
-				(font
-					(size 1.27 1.27)
-				)
-			)
-		)
-		(property "Footprint" "Connector_PinHeader_2.54mm:PinHeader_1x08_P2.54mm_Horizontal"
-			(at 147.32 137.16 0)
-			(effects
-				(font
-					(size 1.27 1.27)
-				)
-				(hide yes)
-			)
-		)
-		(property "Datasheet" "~"
-			(at 147.32 137.16 0)
-			(effects
-				(font
-					(size 1.27 1.27)
-				)
-				(hide yes)
-			)
-		)
-		(property "Description" "Generic connector, single row, 01x08, script generated"
-			(at 147.32 137.16 0)
-			(effects
-				(font
-					(size 1.27 1.27)
-				)
-				(hide yes)
-			)
-		)
-		(pin "1"
-		)
-		(pin "2"
-		)
-		(pin "3"
-		)
-		(pin "4"
-		)
-		(pin "5"
-		)
-		(pin "6"
-		)
-		(pin "7"
-		)
-		(pin "8"
-		)
-		(instances
-			(project "VeloDashboard"
-				(path "/2446985a-a6e1-44ac-a22d-63b6c5e9fbf1"
-					(reference "J3")
-					(unit 1)
-				)
-			)
-		)
-	)
-	(symbol
 		(lib_id "power:GND")
 		(at 55.88 69.85 0)
@@
 					(unit 1)
 				)
+			)
+		)
+	)
+	(symbol
+		(lib_id "Connector:Conn_01x06_Pin")
+		(at 144.78 137.16 90)
+		(unit 1)
+		(exclude_from_sim no)
+		(in_bom yes)
+		(on_board yes)
+		(dnp no)
+		(fields_autoplaced yes)
+		(property "Reference" "J13"
+			(at 146.05 139.7 90)
+			(effects
+				(font
+					(size 1.27 1.27)
+				)
+			)
+		)
+		(property "Value" "To Dashboard"
+			(at 146.05 142.24 90)
+			(effects
+				(font
+					(size 1.27 1.27)
+				)
+			)
+		)
+		(property "Footprint" ""
+			(at 144.78 137.16 0)
+			(effects
+				(font
+					(size 1.27 1.27)
+				)
+				(hide yes)
+			)
+		)
+		(property "Datasheet" "~"
+			(at 144.78 137.16 0)
+			(effects
+				(font
+					(size 1.27 1.27)
+				)
+				(hide yes)
+			)
+		)
+		(property "Description" "Generic connector, single row, 01x06, script generated"
+			(at 144.78 137.16 0)
+			(effects
+				(font
+					(size 1.27 1.27)
+				)
+				(hide yes)
+			)
+		)
+		(pin "1"
+		)
+		(pin "3"
+		)
+		(pin "2"
+		)
+		(pin "4"
+		)
+		(pin "5"
+		)
+		(pin "6"
+		)
+		(instances
+			(project ""
+				(path "/2446985a-a6e1-44ac-a22d-63b6c5e9fbf1"
+					(reference "J13")
+					(unit 1)
+				)
