File: kicad/VeloDashboard/VeloDashboard.kicad_pcb (KiCad board)
At the start: 2 copper layers, 40 parts, among them IC1 LDD-700L, IC2 LDD-700L, IC3 LDD-700L, IC4 LDD-700L, IC5 LDD-700L, IC6 LDD-700L, SW1 On / Off switch, SW2 Left, SW3 Down (lights), SW4 Up (lights), SW5 Brake, SW6 Horn, SW7 Display, SW8 Right, U1 SN74AHCT125N, U2 LC78_05 2.0, U3 Teensy4.0

Commit message: Refacture schematic & raw pcb
Parts:
- removed SW1: On / Off switch, Button_Switch_THT:SW_PUSH-12mm
- added BT1: Battery Cell 3.3V, Battery:Battery_Panasonic_CR2032-HFN_Horizontal_CircularHoles, F.Cu at (14.4, 32.7)
- added J1: OLED, Connector_PinHeader_2.54mm:PinHeader_1x04_P2.54mm_Horizontal, F.Cu at (1.82, 1.82)
- added J1.in1: ~, Connector_PinHeader_2.54mm:PinHeader_1x07_P2.54mm_Horizontal, F.Cu at (38.9, 24.2)
- added J1.out1: Polulu Power, Connector_PinHeader_2.54mm:PinHeader_1x06_P2.54mm_Horizontal, F.Cu at (42.0, 1.82)
- added J2: LED STRIPS, Connector_PinHeader_2.54mm:PinHeader_1x04_P2.54mm_Horizontal, F.Cu at (1.82, 14.1)
- added J3: To Dashboard, Connector_PinHeader_2.54mm:PinHeader_1x08_P2.54mm_Horizontal, F.Cu at (15.2, 1.82)
- added J4: To Computer, Connector_PinHeader_2.54mm:PinHeader_1x08_P2.54mm_Horizontal, F.Cu at (28.6, 1.82)
- added J5: Speed Sensor, Connector_PinHeader_2.54mm:PinHeader_1x03_P2.54mm_Horizontal, F.Cu at (15.2, 53.0)
- added J6: Headlights, Connector_PinHeader_2.54mm:PinHeader_1x04_P2.54mm_Horizontal, F.Cu at (1.82, 26.3)
- added J7: Rearlights, Connector_PinHeader_2.54mm:PinHeader_1x04_P2.54mm_Horizontal, F.Cu at (1.82, 38.6)
- added J8: Blinkers, Connector_PinHeader_2.54mm:PinHeader_1x04_P2.54mm_Horizontal, F.Cu at (1.82, 50.8)
- added J9: PowerSwitch, Connector_PinHeader_2.54mm:PinHeader_1x02_P2.54mm_Horizontal, F.Cu at (15.2, 45.8)
Connections:
- net LED strip 5V renamed +5V
- C1 pad 2: LED strip GND -> GND
- D1 pad 2: LED strip GND -> GND
- D2 pad 2: LED strip GND -> GND
- IC1 pad 4: GND1 -> GND
- IC1 pad 5: FRONT LEFT - -> Net-(IC1--VOUT)
- IC1 pad 6: FRONT LEFT + -> Net-(IC1-+VOUT)
- IC2 pad 4: GND1 -> GND
- IC2 pad 5: FRONT RIGHT - -> Net-(IC2--VOUT)
- IC2 pad 6: FRONT RIGHT + -> Net-(IC2-+VOUT)
- IC3 pad 4: GND1 -> GND
- IC3 pad 5: REAR - -> Net-(IC3--VOUT)
- IC3 pad 6: REAR + -> Net-(IC3-+VOUT)
- IC4 pad 4: GND1 -> GND
- IC4 pad 5: BREAK - -> Net-(IC4--VOUT)
- IC4 pad 6: BREAK + -> Net-(IC4-+VOUT)
- IC5 pad 3: BLINK L -> LED BLINK L
- IC5 pad 4: GND1 -> GND
- IC5 pad 5: BLINK L - -> Net-(IC5--VOUT)
- IC5 pad 6: BLINK L + -> Net-(IC5-+VOUT)
- IC6 pad 3: BLINK R -> LED BLINK R
- IC6 pad 4: GND1 -> GND
- IC6 pad 5: BLINK R - -> Net-(IC6--VOUT)
- IC6 pad 6: BLINK R + -> Net-(IC6-+VOUT)
- R13 pad 1: LED strip GND -> GND
- R14 pad 1: LED strip GND -> GND
- R15 pad 1: LED strip GND -> GND
- R16 pad 1: LED strip GND -> GND
- R19 pad 1: LED strip GND -> GND
- R19 pad 2: BLINK L -> LED BLINK L
- R2 pad 2: LED strip GND -> GND
- R20 pad 1: LED strip GND -> GND
- R20 pad 2: BLINK R -> LED BLINK R
- SW2 pad 2: LED strip GND -> GND
- SW3 pad 2: LED strip GND -> GND
- SW4 pad 2: LED strip GND -> GND
- SW5 pad 2: LED strip GND -> GND
- SW6 pad 2: LED strip GND -> GND
- SW7 pad 2: LED strip GND -> GND
- SW8 pad 2: LED strip GND -> GND
- U1 pad 1: LED strip GND -> GND
- U1 pad 3: LED strip L -> Net-(J2-Pin_1)
- U1 pad 4: LED strip GND -> GND
- U1 pad 6: LED strip R -> Net-(J2-Pin_2)
- U1 pad 7: LED strip GND -> GND
- U2 pad 2: LED strip GND -> GND
- U3 pad 1: LED strip GND -> GND
- U3 pad 14: unconnected-(U3-12_MISO_MQSL-Pad14) -> Power meter
- U3 pad 32: Net-(J3-Pin_8) -> GND
- U3 pad 8: unconnected-(U3-6_OUT1D-Pad8) -> LED BLINK L
- U3 pad 9: Power meter -> LED BLINK R

Commit message: BOM added
Parts:
- added J10: Addon 1, Connector_PinHeader_2.54mm:PinHeader_1x03_P2.54mm_Horizontal, F.Cu at (1.82, 1.82)
- added J11: Addon 2, Connector_PinHeader_2.54mm:PinHeader_1x03_P2.54mm_Horizontal, F.Cu at (1.82, 11.5)
- added J12: extra led strips, Connector_PinHeader_2.54mm:PinHeader_1x04_P2.54mm_Horizontal, F.Cu at (15.2, 18.0)
- added R21: 370, Resistor_THT:R_Axial_DIN0207_L6.3mm_D2.5mm_P10.16mm_Horizontal, F.Cu at (14.5, 1.52)
- added R22: 370, Resistor_THT:R_Axial_DIN0207_L6.3mm_D2.5mm_P10.16mm_Horizontal, F.Cu at (14.5, 5.58)
- added R23: 370, Resistor_THT:R_Axial_DIN0207_L6.3mm_D2.5mm_P10.16mm_Horizontal, F.Cu at (14.5, 9.62)
- added R24: 370, Resistor_THT:R_Axial_DIN0207_L6.3mm_D2.5mm_P10.16mm_Horizontal, F.Cu at (14.5, 13.7)
Connections:
- R3 pad 2: Net-(U3-20_A6_TX5_LRCLK1) -> Net-(U3-21_A7_RX5_BCLK1)
- R4 pad 1: Net-(U3-19_A5_SCL0) -> Net-(U3-20_A6_TX5_LRCLK1)
- R5 pad 1: Net-(U3-18_A4_SDA0) -> Net-(U3-19_A5_SCL0)
- U1 pad 10: unconnected-(U1-3~{OE}-Pad10) -> GND
- U1 pad 11: unconnected-(U1-4Y-Pad11) -> Net-(U1-4Y)
- U1 pad 12: unconnected-(U1-4A-Pad12) -> Net-(U1-4A)
- U1 pad 13: unconnected-(U1-4~{OE}-Pad13) -> GND
- U1 pad 3: Net-(J2-Pin_1) -> Net-(U1-1Y)
- U1 pad 6: Net-(J2-Pin_2) -> Net-(U1-2Y)
- U1 pad 8: unconnected-(U1-3Y-Pad8) -> Net-(U1-3Y)
- U1 pad 9: unconnected-(U1-3A-Pad9) -> Net-(U1-3A)
- U3 pad 14: Power meter -> unconnected-(U3-12_MISO_MQSL-Pad14)
- U3 pad 2: unconnected-(U3-0_RX1_CRX2_CS1-Pad2) -> Net-(U1-3A)
- U3 pad 21: unconnected-(U3-14_A0_TX3_SPDIF_OUT-Pad21) -> Addon 1
- U3 pad 22: unconnected-(U3-15_A1_RX3_SPDIF_IN-Pad22) -> Addon 2
- U3 pad 25: Net-(U3-18_A4_SDA0) -> Power meter
- U3 pad 28: unconnected-(U3-21_A7_RX5_BCLK1-Pad28) -> Net-(U3-21_A7_RX5_BCLK1)
- U3 pad 3: unconnected-(U3-1_TX1_CTX2_MISO1-Pad3) -> Net-(U1-4A)

Commit message: refacture due to soldering
Parts:
- J10: value Addon 1 -> Cadans sensor
Connections:
- J10 pad 2: Addon 1 -> Cadans
- J11 pad 2: Addon 2 -> Addon
- J3 pad 4: unconnected-(J3-Pin_4-Pad4) -> Net-(J3-Pin_4)
- J3 pad 6: Net-(J3-Pin_6) -> unconnected-(J3-Pin_6-Pad6)
- J4 pad 1: Net-(J4-Pin_1) -> Net-(D2-K)
- J4 pad 2: Net-(J4-Pin_2) -> Net-(D1-K)
- J4 pad 4: unconnected-(J4-Pin_4-Pad4) -> Net-(J4-Pin_4)
- J4 pad 5: Net-(D2-K) -> Net-(J4-Pin_5)
- J4 pad 6: Net-(D1-K) -> Net-(J4-Pin_5)
- J4 pad 7: unconnected-(J4-Pin_7-Pad7) -> GND
- J5 pad 2: Net-(J5-Pin_2) -> Speed
- R10 pad 1: Net-(U3-23_A9_CRX1_MCLK1) -> Net-(U3-20_A6_TX5_LRCLK1)
- R10 pad 2: Net-(J3-Pin_6) -> Net-(J3-Pin_2)
- R11 pad 1: Net-(J4-Pin_3) -> Net-(J4-Pin_4)
- R18 pad 2: Net-(J4-Pin_1) -> Net-(J4-Pin_3)
- R3 pad 1: Net-(J3-Pin_3) -> Net-(J3-Pin_4)
- R3 pad 2: Net-(U3-21_A7_RX5_BCLK1) -> Net-(U3-23_A9_CRX1_MCLK1)
- R4 pad 1: Net-(U3-20_A6_TX5_LRCLK1) -> Net-(U3-22_A8_CTX1)
- R4 pad 2: Net-(J3-Pin_2) -> Net-(J3-Pin_5)
- R5 pad 1: Net-(U3-19_A5_SCL0) -> Net-(J3-Pin_3)
- R5 pad 2: Net-(J3-Pin_1) -> Net-(U3-21_A7_RX5_BCLK1)
- R6 pad 1: Net-(J3-Pin_1) -> Net-(J3-Pin_3)
- R7 pad 1: Net-(J3-Pin_2) -> Net-(J3-Pin_4)
- R8 pad 1: Net-(J3-Pin_3) -> Net-(J3-Pin_5)
- R9 pad 1: Net-(U3-22_A8_CTX1) -> Net-(U3-19_A5_SCL0)
- R9 pad 2: Net-(J3-Pin_5) -> Net-(J3-Pin_1)
- SW2 pad 1: Net-(J4-Pin_3) -> Net-(J4-Pin_4)
- SW5 pad 1: Net-(J4-Pin_2) -> Net-(J4-Pin_5)
- SW8 pad 1: Net-(J4-Pin_1) -> Net-(J4-Pin_3)
- U3 pad 10: LED front L -> LED rear
- U3 pad 11: LED front R -> LED break
- U3 pad 12: LED rear -> LED front L
- U3 pad 13: LED break -> LED front R
- U3 pad 21: Addon 1 -> Speed
- U3 pad 22: Addon 2 -> Cadans
- U3 pad 6: Net-(J5-Pin_2) -> Addon
Changed lines of the file:
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@@
 	(net 28 "Net-(J3-Pin_2)")
 	(net 29 "Net-(U3-19_A5_SCL0)")
-	(net 30 "Addon 1")
+	(net 30 "unconnected-(J3-Pin_6-Pad6)")
 	(net 31 "Net-(J3-Pin_1)")
 	(net 32 "+3.3V")
 	(net 33 "Net-(U3-22_A8_CTX1)")
 	(net 34 "Net-(J3-Pin_5)")
-	(net 35 "Net-(J3-Pin_6)")
+	(net 35 "Net-(J3-Pin_4)")
 	(net 36 "Net-(U3-23_A9_CRX1_MCLK1)")
 	(net 37 "Net-(J4-Pin_3)")
@@
 	(net 40 "Net-(R17-Pad1)")
 	(net 41 "Net-(R17-Pad2)")
-	(net 42 "Net-(J4-Pin_1)")
+	(net 42 "Net-(J4-Pin_4)")
 	(net 43 "Net-(J1.out1-Pin_6)")
 	(net 44 "Net-(J1.out1-Pin_5)")
-	(net 45 "Net-(J4-Pin_2)")
-	(net 46 "Addon 2")
+	(net 45 "Net-(J4-Pin_5)")
+	(net 46 "Speed")
 	(net 47 "Net-(J12-Pin_1)")
-	(net 48 "Net-(J5-Pin_2)")
+	(net 48 "Cadans")
 	(net 49 "Net-(U1-1A)")
 	(net 50 "Net-(U1-2A)")
@@
 	(net 94 "unconnected-(J1.in1-Pin_5-Pad5)")
 	(net 95 "unconnected-(J3-Pin_7-Pad7)")
-	(net 96 "unconnected-(J3-Pin_4-Pad4)")
-	(net 97 "unconnected-(J4-Pin_4-Pad4)")
-	(net 98 "unconnected-(J4-Pin_7-Pad7)")
+	(net 96 "Addon")
 	(footprint "Connector_PinHeader_2.54mm:PinHeader_1x04_P2.54mm_Horizontal"
 		(layer "F.Cu")
@@
 			(layers "*.Cu" "*.Mask")
 			(remove_unused_layers no)
-			(net 26 "Net-(U3-20_A6_TX5_LRCLK1)")
+			(net 33 "Net-(U3-22_A8_CTX1)")
 			(pintype "passive")
 		)
@@
 			(layers "*.Cu" "*.Mask")
 			(remove_unused_layers no)
-			(net 28 "Net-(J3-Pin_2)")
+			(net 34 "Net-(J3-Pin_5)")
 			(pintype "passive")
 		)
@@
 			(layers "*.Cu" "*.Mask")
 			(remove_unused_layers no)
-			(net 27 "Net-(J3-Pin_3)")
+			(net 34 "Net-(J3-Pin_5)")
 			(pintype "passive")
 		)
@@
 			(layers "*.Cu" "*.Mask")
 			(remove_unused_layers no)
-			(net 42 "Net-(J4-Pin_1)")
+			(net 4 "Net-(D2-K)")
 			(pinfunction "Pin_1")
 			(pintype "passive")
@@
 			(layers "*.Cu" "*.Mask")
 			(remove_unused_layers no)
-			(net 45 "Net-(J4-Pin_2)")
+			(net 3 "Net-(D1-K)")
 			(pinfunction "Pin_2")
 			(pintype "passive")
@@
 			(layers "*.Cu" "*.Mask")
 			(remove_unused_layers no)
-			(net 97 "unconnected-(J4-Pin_4-Pad4)")
+			(net 42 "Net-(J4-Pin_4)")
 			(pinfunction "Pin_4")
-			(pintype "passive+no_connect")
+			(pintype "passive")
 		)
 		(pad "5" thru_hole oval
@@
 			(layers "*.Cu" "*.Mask")
 			(remove_unused_layers no)
-			(net 4 "Net-(D2-K)")
+			(net 45 "Net-(J4-Pin_5)")
 			(pinfunction "Pin_5")
 			(pintype "passive")
@@
 			(layers "*.Cu" "*.Mask")
 			(remove_unused_layers no)
-			(net 3 "Net-(D1-K)")
+			(net 45 "Net-(J4-Pin_5)")
 			(pinfunction "Pin_6")
 			(pintype "passive")
@@
 			(layers "*.Cu" "*.Mask")
 			(remove_unused_layers no)
-			(net 98 "unconnected-(J4-Pin_7-Pad7)")
+			(net 1 "GND")
 			(pinfunction "Pin_7")
-			(pintype "passive+no_connect")
+			(pintype "passive")
 		)
 		(pad "8" thru_hole oval
@@
 			(layers "*.Cu" "*.Mask")
 			(remove_unused_layers no)
-			(net 42 "Net-(J4-Pin_1)")
+			(net 37 "Net-(J4-Pin_3)")
 			(pinfunction "1")
 			(pintype "passive")
@@
 			(layers "*.Cu" "*.Mask")
 			(remove_unused_layers no)
-			(net 42 "Net-(J4-Pin_1)")
+			(net 37 "Net-(J4-Pin_3)")
 			(pinfunction "1")
 			(pintype "passive")
@@
 			(layers "*.Cu" "*.Mask")
 			(remove_unused_layers no)
-			(net 46 "Addon 2")
+			(net 96 "Addon")
 			(pinfunction "Pin_2")
 			(pintype "passive")
@@
 			(layers "*.Cu" "*.Mask")
 			(remove_unused_layers no)
-			(net 96 "unconnected-(J3-Pin_4-Pad4)")
+			(net 35 "Net-(J3-Pin_4)")
 			(pinfunction "Pin_4")
-			(pintype "passive+no_connect")
+			(pintype "passive")
 		)
 		(pad "5" thru_hole oval
@@
 			(layers "*.Cu" "*.Mask")
 			(remove_unused_layers no)
-			(net 35 "Net-(J3-Pin_6)")
+			(net 30 "unconnected-(J3-Pin_6-Pad6)")
 			(pinfunction "Pin_6")
-			(pintype "passive")
+			(pintype "passive+no_connect")
 		)
 		(pad "7" thru_hole oval
@@
 		(fp_arc
 			(start 20.68 -1.32)
-			(mid 21.329556 -0.950479)
+			(mid 21.329538 -0.95046)
 			(end 21.59 -0.25)
 			(stroke
@@
 			(layers "*.Cu" "*.Mask")
 			(remove_unused_layers no)
-			(net 33 "Net-(U3-22_A8_CTX1)")
+			(net 29 "Net-(U3-19_A5_SCL0)")
 			(pintype "passive")
 		)
@@
 			(layers "*.Cu" "*.Mask")
 			(remove_unused_layers no)
-			(net 34 "Net-(J3-Pin_5)")
+			(net 31 "Net-(J3-Pin_1)")
 			(pintype "passive")
 		)
@@
 			(layers "*.Cu" "*.Mask")
 			(remove_unused_layers no)
-			(net 36 "Net-(U3-23_A9_CRX1_MCLK1)")
+			(net 26 "Net-(U3-20_A6_TX5_LRCLK1)")
 			(pintype "passive")
 		)
@@
 			(layers "*.Cu" "*.Mask")
 			(remove_unused_layers no)
-			(net 35 "Net-(J3-Pin_6)")
+			(net 28 "Net-(J3-Pin_2)")
 			(pintype "passive")
 		)
@@
 			(layers "*.Cu" "*.Mask")
 			(remove_unused_layers no)
-			(net 48 "Net-(J5-Pin_2)")
+			(net 96 "Addon")
 			(pinfunction "4_BCLK2")
 			(pintype "bidirectional")
@@
 			(layers "*.Cu" "*.Mask")
 			(remove_unused_layers no)
-			(net 7 "LED front L")
+			(net 15 "LED rear")
 			(pinfunction "8_TX2_IN1")
 			(pintype "bidirectional")
@@
 			(layers "*.Cu" "*.Mask")
 			(remove_unused_layers no)
-			(net 10 "LED front R")
+			(net 17 "LED break")
 			(pinfunction "9_OUT1C")
 			(pintype "bidirectional")
@@
 			(layers "*.Cu" "*.Mask")
 			(remove_unused_layers no)
-			(net 15 "LED rear")
+			(net 7 "LED front L")
 			(pinfunction "10_CS_MQSR")
 			(pintype "bidirectional")
@@
 			(layers "*.Cu" "*.Mask")
 			(remove_unused_layers no)
-			(net 17 "LED break")
+			(net 10 "LED front R")
 			(pinfunction "11_MOSI_CTX1")
 			(pintype "bidirectional")
@@
 			(layers "*.Cu" "*.Mask")
 			(remove_unused_layers no)
-			(net 30 "Addon 1")
+			(net 46 "Speed")
 			(pinfunction "14_A0_TX3_SPDIF_OUT")
 			(pintype "bidirectional")
@@
 			(layers "*.Cu" "*.Mask")
 			(remove_unused_layers no)
-			(net 46 "Addon 2")
+			(net 48 "Cadans")
 			(pinfunction "15_A1_RX3_SPDIF_IN")
 			(pintype "bidirectional")
@@
 			(layers "*.Cu" "*.Mask")
 			(remove_unused_layers no)
-			(net 31 "Net-(J3-Pin_1)")
+			(net 27 "Net-(J3-Pin_3)")
 			(pintype "passive")
 		)
@@
 			(layers "*.Cu" "*.Mask")
 			(remove_unused_layers no)
-			(net 45 "Net-(J4-Pin_2)")
+			(net 45 "Net-(J4-Pin_5)")
 			(pinfunction "1")
 			(pintype "passive")
@@
 			(layers "*.Cu" "*.Mask")
 			(remove_unused_layers no)
-			(net 45 "Net-(J4-Pin_2)")
+			(net 45 "Net-(J4-Pin_5)")
 			(pinfunction "1")
 			(pintype "passive")
@@
 			(layers "*.Cu" "*.Mask")
 			(remove_unused_layers no)
-			(net 37 "Net-(J4-Pin_3)")
+			(net 42 "Net-(J4-Pin_4)")
 			(pinfunction "1")
 			(pintype "passive")
@@
 			(layers "*.Cu" "*.Mask")
 			(remove_unused_layers no)
-			(net 37 "Net-(J4-Pin_3)")
+			(net 42 "Net-(J4-Pin_4)")
 			(pinfunction "1")
 			(pintype "passive")
@@
 			(layers "*.Cu" "*.Mask")
 			(remove_unused_layers no)
-			(net 29 "Net-(U3-19_A5_SCL0)")
+			(net 27 "Net-(J3-Pin_3)")
 			(pintype "passive")
 		)
@@
 			(layers "*.Cu" "*.Mask")
 			(remove_unused_layers no)
-			(net 31 "Net-(J3-Pin_1)")
+			(net 52 "Net-(U3-21_A7_RX5_BCLK1)")
 			(pintype "passive")
 		)
@@
 			(layers "*.Cu" "*.Mask")
 			(remove_unused_layers no)
-			(net 27 "Net-(J3-Pin_3)")
+			(net 35 "Net-(J3-Pin_4)")
 			(pintype "passive")
 		)
@@
 			(layers "*.Cu" "*.Mask")
 			(remove_unused_layers no)
-			(net 52 "Net-(U3-21_A7_RX5_BCLK1)")
+			(net 36 "Net-(U3-23_A9_CRX1_MCLK1)")
 			(pintype "passive")
 		)
@@
 			(layers "*.Cu" "*.Mask")
 			(remove_unused_layers no)
-			(net 37 "Net-(J4-Pin_3)")
+			(net 42 "Net-(J4-Pin_4)")
 			(pintype "passive")
 		)
@@
 			(layers "*.Cu" "*.Mask")
 			(remove_unused_layers no)
-			(net 28 "Net-(J3-Pin_2)")
+			(net 35 "Net-(J3-Pin_4)")
 			(pintype "passive")
 		)
@@
 			(layers "*.Cu" "*.Mask")
 			(remove_unused_layers no)
-			(net 48 "Net-(J5-Pin_2)")
+			(net 46 "Speed")
 			(pinfunction "Pin_2")
 			(pintype "passive")
@@
 			)
 		)
-		(property "Value" "Addon 1"
+		(property "Value" "Cadans sensor"
 			(at 4.385 7.35 0)
 			(layer "F.Fab")
@@
 			(layers "*.Cu" "*.Mask")
 			(remove_unused_layers no)
-			(net 30 "Addon 1")
+			(net 48 "Cadans")
 			(pinfunction "Pin_2")
 			(pintype "passive")
@@
 			(layers "*.Cu" "*.Mask")
 			(remove_unused_layers no)
-			(net 42 "Net-(J4-Pin_1)")
+			(net 37 "Net-(J4-Pin_3)")
 			(pintype "passive")
 		)
